Commit message: Small fixes, added Tetrapod Gait and corrected Realsense camera origin in URDF

File: robot/shelob_syropod.urdf (robot description, URDF)
Before this commit: robot shelob_model, 36 links, 35 joints
Joints:
- joint vision_joint: origin xyz=0.1175 0.0174 0.0336 rpy=0.0000 1.4661 0.0000 -> xyz=0.1175 0.0174 0.0336 rpy=-1.4661 0.0000 -1.5708

Commit message: Removed ASC code. Added Abdomen joint/link. TODO write code to manipulate.

File: robot/shelob_syropod.urdf (robot description, URDF)
Before this commit: robot shelob_model, 36 links, 35 joints
Joints:
- joint AL_tarsus_joint: limit lower=-1.6779 upper=0.6045 effort=1.9 velocity=2.35619449 -> lower=-1.6779 upper=1.5710 effort=1.9 velocity=2.35619449
- joint AL_tibia_joint: limit lower=-2.2422 upper=0.0960 effort=1.9 velocity=2.35619449 -> lower=-2.2422 upper=1.5710 effort=1.9 velocity=2.35619449
- joint AR_tarsus_joint: limit lower=-1.6779 upper=0.6045 effort=1.9 velocity=2.35619449 -> lower=-1.6779 upper=1.5710 effort=1.9 velocity=2.35619449
- joint AR_tibia_joint: limit lower=-2.2422 upper=0.0960 effort=1.9 velocity=2.35619449 -> lower=-2.2422 upper=1.5710 effort=1.9 velocity=2.35619449
- joint BL_tarsus_joint: limit lower=-1.6779 upper=0.6045 effort=1.9 velocity=2.35619449 -> lower=-1.6779 upper=1.5710 effort=1.9 velocity=2.35619449
- joint BL_tibia_joint: limit lower=-2.2422 upper=0.0960 effort=1.9 velocity=2.35619449 -> lower=-2.2422 upper=1.5710 effort=1.9 velocity=2.35619449
- joint BR_tarsus_joint: limit lower=-1.6779 upper=0.6045 effort=1.9 velocity=2.35619449 -> lower=-1.6779 upper=1.5710 effort=1.9 velocity=2.35619449
- joint BR_tibia_joint: limit lower=-2.2422 upper=0.0960 effort=1.9 velocity=2.35619449 -> lower=-2.2422 upper=1.5710 effort=1.9 velocity=2.35619449
- joint CL_tarsus_joint: limit lower=-1.6779 upper=0.6045 effort=1.9 velocity=2.35619449 -> lower=-1.6779 upper=1.5710 effort=1.9 velocity=2.35619449
- joint CL_tibia_joint: limit lower=-2.2422 upper=0.0960 effort=1.9 velocity=2.35619449 -> lower=-2.2422 upper=1.5710 effort=1.9 velocity=2.35619449
- joint CR_tarsus_joint: limit lower=-1.6779 upper=0.6045 effort=1.9 velocity=2.35619449 -> lower=-1.6779 upper=1.5710 effort=1.9 velocity=2.35619449
- joint CR_tibia_joint: limit lower=-2.2422 upper=0.0960 effort=1.9 velocity=2.35619449 -> lower=-2.2422 upper=1.5710 effort=1.9 velocity=2.35619449
- joint DL_tarsus_joint: limit lower=-1.6779 upper=0.6045 effort=1.9 velocity=2.35619449 -> lower=-1.6779 upper=1.5710 effort=1.9 velocity=2.35619449
- joint DL_tibia_joint: limit lower=-2.2422 upper=0.0960 effort=1.9 velocity=2.35619449 -> lower=-2.2422 upper=1.5710 effort=1.9 velocity=2.35619449
- joint DR_tarsus_joint: limit lower=-1.6779 upper=0.6045 effort=1.9 velocity=2.35619449 -> lower=-1.6779 upper=1.5710 effort=1.9 velocity=2.35619449
- joint DR_tibia_joint: limit lower=-2.2422 upper=0.0960 effort=1.9 velocity=2.35619449 -> lower=-2.2422 upper=1.5710 effort=1.9 velocity=2.35619449
